Commit message: add control plugin argument

File: ur_gazebo/urdf/ur_macro.xacro (robot description, xacro)
@@ -31,5 +31,6 @@
   -->
   <!-- Definition of the main macro -->
-  <xacro:macro name="ur_robot_gazebo" params="
+  <xacro:macro name="ur_robot_gazebo"
+    params="
    prefix
    joint_limits_parameters_file
@@ -38,5 +39,6 @@
    visual_parameters_file
    transmission_hw_interface:=hardware_interface/EffortJointInterface
-   safety_limits:=false safety_pos_margin:=0.15 safety_k_position:=20"
+   safety_limits:=false safety_pos_margin:=0.15 safety_k_position:=20
+   load_gazebo_ros_control_plugin:=true"
   >
     <!--
@@ -46,5 +48,5 @@
       the definitions for the real robot.
     -->
-  <xacro:include filename="$(find ur_description)/urdf/inc/ur_macro.xacro"/>
+    <xacro:include filename="$(find ur_description)/urdf/inc/ur_macro.xacro" />
     <!-- Instantiate model for the REAL robot. -->
     <xacro:ur_robot
@@ -85,10 +87,12 @@
       controllers to control the virtual robot hw.
     -->
-    <gazebo>
-      <plugin name="ros_control" filename="libgazebo_ros_control.so">
-        <!--robotNamespace>/</robotNamespace-->
-        <!--robotSimType>gazebo_ros_control/DefaultRobotHWSim</robotSimType-->
-      </plugin>
-    </gazebo>
+    <xacro:if value="${load_gazebo_ros_control_plugin}">
+      <gazebo>
+        <plugin name="ros_control" filename="libgazebo_ros_control.so">
+          <!--robotNamespace>/</robotNamespace-->
+          <!--robotSimType>gazebo_ros_control/DefaultRobotHWSim</robotSimType-->
+        </plugin>
+      </gazebo>
+    </xacro:if>
   </xacro:macro>
 </robot>
